File: ergogen/output/pcbs/mr_useful.kicad_pcb (KiCad board)
At the start: 2 copper layers, 57 x 95 mm, 36 parts

Commit message: Fix net definitions
Parts:
- removed ?: , Seeeduino XIAO-MOUDLE14P-2.54-21X17.8MM tht maybe
- added MCU1: , Seeeduino XIAO-MOUDLE14P-2.54-21X17.8MM tht maybe, B.Cu at (79.0, 49.0)
- moved D3 36.1 mm to (85.3, 110.3)
- moved LED11 26.9 mm to (60.0, 115.5)
- moved LED12 26.9 mm to (79.0, 96.5)
- moved LED3 26.9 mm to (79.0, 101.2)
- moved S3 26.9 mm to (79.0, 106.0)
- moved D2 22.3 mm to (85.3, 129.3)
- moved LED1 19.0 mm to (60.0, 120.2)
- moved LED2 19.0 mm to (79.0, 120.2)
- moved S1 19.0 mm to (60.0, 125.0)
- moved S2 19.0 mm to (79.0, 125.0)
- moved D5 11.7 mm to (66.3, 72.3)
- moved D6 11.7 mm to (66.3, 53.4)
- moved D10 11.7 mm to (104.3, 53.4)
- moved D4 11.7 mm to (104.3, 129.3)
- moved D7 11.7 mm to (85.3, 72.3)
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Connections:
- net right_default renamed right_down
- D1 pad 2: middle_down -> left_down
- D2 pad 1: R1 -> R0
- D2 pad 2: middle_up -> middle_down
- D3 pad 1: (no net) -> R1
- D3 pad 2: left_default -> middle_up
- D4 pad 1: (no net) -> R0
- LED1 pad 2: LED_5 -> LED_4
- LED1 pad 4: LED_4 -> LED_3
- LED11 pad 1: VCC -> RAW
- LED11 pad 2: ULED_2 -> ULED_3
- LED11 pad 4: ULED_1 -> ULED_2
- LED12 pad 1: VCC -> RAW
- LED12 pad 2: (no net) -> ULED_2
- LED12 pad 4: (no net) -> ULED_1
- LED13 pad 1: VCC -> RAW
- LED13 pad 2: (no net) -> ULED_1
- LED13 pad 4: (no net) -> LED_10
- LED14 pad 1: VCC -> RAW
- LED15 pad 1: VCC -> RAW
- LED2 pad 2: LED_6 -> LED_5
- LED2 pad 4: LED_5 -> LED_4
- LED3 pad 2: (no net) -> LED_6
- LED3 pad 4: (no net) -> LED_5
- LED4 pad 2: (no net) -> LED_10
- LED4 pad 4: (no net) -> LED_9
- S1 pad 1: C1 -> C0
- S1 pad 2: middle_down -> left_down
- S2 pad 2: middle_up -> middle_down
- S3 pad 1: C0 -> C1
- S3 pad 2: left_default -> middle_up

Commit message: Fix VCC net name and generate outputs
Parts:
- moved D1 4.50 mm to (62.2, 131.0), turned to 0 degrees
- moved D2 4.50 mm to (81.2, 131.0), turned to 0 degrees
- moved D3 4.50 mm to (81.2, 112.0), turned to 0 degrees
- moved D4 4.50 mm to (100.2, 131.0), turned to 0 degrees
- moved D5 4.50 mm to (62.2, 74.0), turned to 0 degrees
- moved D7 4.50 mm to (81.2, 74.0), turned to 0 degrees
- moved D9 4.50 mm to (100.2, 74.0), turned to 0 degrees
- moved D10 4.50 mm to (100.2, 55.0), turned to 0 degrees
- moved D6 4.50 mm to (62.2, 55.0), turned to 0 degrees
- moved D8 4.50 mm to (81.2, 55.0), turned to 0 degrees
Connections:
- LED11 pad 1: RAW -> VCC
- LED12 pad 1: RAW -> VCC
- LED13 pad 1: RAW -> VCC
- LED14 pad 1: RAW -> VCC
- LED15 pad 1: RAW -> VCC
- MCU1 pad 3V3: RAW3V3 -> VCC
- MCU1 pad P0: LED -> P0
- MCU1 pad P3: P3 -> LED
- MCU1 pad RAW: RAW5V -> RAW

Commit message: Update diode footprint to be on one side only
Parts:
- D1, D10, D2, D3, D4, D5, D6, D7, D8, D9: moved to B.Cu
