File: ergogen/output/pcbs/mr_useful_routed.kicad_pcb (KiCad board)
At the start: 2 copper layers, 57 x 95 mm, 36 parts

Commit message: Update diode footprint to be on one side only
Parts:
- D1, D10, D2, D3, D4, D5, D6, D7, D8, D9: moved to B.Cu
Routing:
- net R3: track 78.4 -> 58.9 mm, vias 4 -> 1
- net VCC: track 272.7 -> 288.3 mm, vias 0 -> 2
- net R4: track 58.7 -> 43.3 mm, vias 4 -> 0
- net R0: track 131.6 -> 121.2 mm, vias 3 -> 1
- net GND: track 299.4 -> 309.5 mm
- net ULED_4: track 50.8 -> 57.7 mm
- net R1: track 72.4 -> 66.5 mm
- net LED_6: track 46.3 -> 51.6 mm, vias 0 -> 2
- net left_down: track 6.92 -> 11.3 mm
- net ULED_2: track 31.2 -> 26.9 mm, vias 2 -> 0
- net third_top: track 6.92 -> 3.46 mm
- net second_top: track 6.92 -> 3.46 mm
- net first_top: track 6.92 -> 3.46 mm
- net third_bottom: track 6.92 -> 3.46 mm
- net second_bottom: track 6.92 -> 3.46 mm
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
Commit message: Add logo and reference
Parts:
- added LOGO1: , logo_mr_useful, F.Cu at (79.0, 87.0)
Changed lines of the file:
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@@
     (tracks 418)
     (zones 0)
-    (modules 36)
+    (modules 37)
     (nets 42)
   )
@@
       (net 36 P0))
   )
+  (module logo_mr_useful (layer F.Cu)
+    (at 79 87)
+    (fp_text reference LOGO1 (at 0 0) (layer F.SilkS) hide
+      (effects (font (size 1.27 1.27) (thickness 0.15)))
+    )
+    (fp_text value "" (at 0 0) (layer F.SilkS) hide
+      (effects (font (size 1.27 1.27) (thickness 0.15)))
+    )
+    (fp_text user github.com/ceoloide/mr_useful (at 0 1) (layer F.SilkS)
+      (effects (font (size 1 1) (thickness 0.1)) (justify bottom))
+    )
+    (fp_text user "v0.1 pre-release" (at 0 3) (layer F.SilkS)
+      (effects (font (size 1 1) (thickness 0.1)) (justify bottom))
+    )
+    (fp_poly (pts (xy 2.972094 -3.801687) (xy 3.678531 -3.801687) (xy 3.654719 -4.079996) (xy 3.591219 -4.264047)
+      (xy 3.341188 -4.400969) (xy 3.185414 -4.368226) (xy 3.075281 -4.27) (xy 3.005828 -4.087437)
+      (xy 2.972094 -3.801687)) (layer F.SilkS) (width 0.01))
+    (fp_poly (pts (xy -9.485812 -6.37476) (xy -10.312635 -6.37476) (xy -10.539555 -6.363612) (xy -10.76429 -6.330276)
+      (xy -10.984675 -6.275073) (xy -11.198587 -6.198533) (xy -11.403968 -6.101396) (xy -11.598838 -5.984595)
+      (xy -11.781322 -5.849256) (xy -11.949661 -5.696682) (xy -12.102235 -5.528343) (xy -12.237574 -5.345859)
+      (xy -12.354375 -5.150989) (xy -12.451513 -4.945608) (xy -12.528052 -4.731695) (xy -12.583255 -4.51131)
+      (xy -12.616592 -4.286576) (xy -12.627739 -4.059656) (xy -12.616592 -3.832736) (xy -12.583255 -3.608002)
+      (xy -12.528052 -3.387617) (xy -12.451513 -3.173704) (xy -12.354375 -2.968323) (xy -12.237574 -2.773453)
+      (xy -12.102235 -2.590969) (xy -11.949661 -2.42263) (xy -11.781322 -2.270056) (xy -11.598838 -2.134717)
+      (xy -11.403968 -2.017916) (xy -11.198587 -1.920779) (xy -10.984675 -1.844239) (xy -10.76429 -1.789036)
+      (xy -10.539555 -1.7557) (xy -10.312635 -1.744552) (xy -9.485812 -1.744552) (xy -9.096875 -1.744552)
+      (xy -9.096875 -2.611062) (xy -9.485812 -2.611062) (xy -9.335 -5.50825) (xy -8.815094 -5.50825)
+      (xy -8.573 -3.662781) (xy -8.565062 -3.662781) (xy -8.326937 -5.50825) (xy -7.826875 -5.50825)
+      (xy -7.680031 -2.611062) (xy -8.104687 -2.611062) (xy -8.164219 -5.071687) (xy -8.168187 -5.071687)
+      (xy -8.41425 -3.28575) (xy -8.791281 -3.28575) (xy -9.0175 -5.071687) (xy -9.029406 -5.071687)
+      (xy -9.096875 -2.611062) (xy -9.096875 -1.744552) (xy -6.767219 -1.744552) (xy -6.767219 -2.611062)
+      (xy -7.203781 -2.611062) (xy -7.203781 -4.508125) (xy -6.950734 -4.58242) (xy -6.693241 -4.640205)
+      (xy -6.431304 -4.68148) (xy -6.164921 -4.706245) (xy -5.894094 -4.7145) (xy -5.894094 -4.385094)
+      (xy -6.197924 -4.372305) (xy -6.490288 -4.333941) (xy -6.771187 -4.27) (xy -6.767219 -2.611062)
+      (xy -6.767219 -1.744552) (xy -4.92175 -1.744552) (xy -4.92175 -2.611062) (xy -4.92175 -3.28575)
+      (xy -4.28675 -3.28575) (xy -4.28675 -2.611062) (xy -4.92175 -2.611062) (xy -4.92175 -1.744552)
+      (xy -0.643437 -1.744552) (xy -0.643437 -2.571375) (xy -0.899863 -2.591659) (xy -1.10293 -2.652514)
+      (xy -1.252641 -2.753937) (xy -1.355167 -2.902986) (xy -1.416682 -3.106715) (xy -1.437187 -3.365125)
+      (xy -1.437187 -5.50825) (xy -0.988719 -5.50825) (xy -0.988719 -3.4445) (xy -0.968875 -3.187523)
+      (xy -0.909344 -3.027781) (xy -0.801195 -2.944437) (xy -0.6355 -2.916656) (xy -0.361656 -3.025797)
+      (xy -0.302125 -3.185043) (xy -0.282281 -3.4445) (xy -0.282281 -5.50825) (xy 0.150313 -5.50825)
+      (xy 0.150313 -3.365125) (xy 0.129807 -3.106715) (xy 0.068292 -2.902986) (xy -0.034234 -2.753937)
+      (xy -0.183944 -2.652514) (xy -0.387012 -2.591659) (xy -0.643437 -2.571375) (xy -0.643437 -1.744552)
+      (xy 1.317125 -1.744552) (xy 1.317125 -2.571375) (xy 1.073708 -2.585486) (xy 0.846167 -2.627819)
+      (xy 0.6345 -2.698375) (xy 0.6345 -3.047625) (xy 0.951008 -2.931539) (xy 1.249656 -2.892843)
+      (xy 1.551281 -2.958328) (xy 1.642563 -3.166687) (xy 1.571125 -3.365125) (xy 1.309188 -3.484187)
+      (xy 0.986727 -3.593824) (xy 0.773406 -3.732234) (xy 0.654344 -3.910332) (xy 0.614656 -4.139031)
+      (xy 0.661289 -4.384597) (xy 0.801188 -4.565672) (xy 1.033359 -4.677293) (xy 1.356813 -4.7145)
+      (xy 1.588764 -4.704798) (xy 1.808368 -4.675694) (xy 2.015625 -4.627187) (xy 2.015625 -4.297781)
+      (xy 1.698125 -4.372195) (xy 1.3965 -4.397) (xy 1.137539 -4.332508) (xy 1.051219 -4.139031)
+      (xy 1.120672 -3.960437) (xy 1.356813 -3.849312) (xy 1.710527 -3.738187) (xy 1.930297 -3.60325)
+      (xy 2.044895 -3.420687) (xy 2.083094 -3.166687) (xy 2.032988 -2.913679) (xy 1.882672 -2.726156)
+      (xy 1.641074 -2.61007) (xy 1.317125 -2.571375) (xy 1.317125 -1.744552) (xy 3.432469 -1.744552)
+      (xy 3.432469 -2.571375) (xy 3.153554 -2.60114) (xy 2.925351 -2.690437) (xy 2.747859 -2.839265)
+      (xy 2.62108 -3.047625) (xy 2.545012 -3.315515) (xy 2.519656 -3.642937) (xy 2.542807 -3.970359)
+      (xy 2.612261 -4.23825) (xy 2.728016 -4.446609) (xy 2.890073 -4.595437) (xy 3.098432 -4.684734)
+      (xy 3.353094 -4.7145) (xy 3.585486 -4.686498) (xy 3.774663 -4.602493) (xy 3.920625 -4.462484)
+      (xy 4.024254 -4.260298) (xy 4.086431 -3.989762) (xy 4.107156 -3.650875) (xy 4.099219 -3.492125)
+      (xy 2.972094 -3.492125) (xy 3.018231 -3.213816) (xy 3.116953 -3.029765) (xy 3.271238 -2.927074)
+      (xy 3.484063 -2.892843) (xy 3.728141 -2.919633) (xy 4 -3) (xy 4 -2.670593)
+      (xy 3.709289 -2.596179) (xy 3.432469 -2.571375) (xy 3.432469 -1.744552) (xy 5.456531 -1.744552)
+      (xy 5.456531 -2.611062) (xy 5.019969 -2.611062) (xy 5.019969 -4.273969) (xy 4.583406 -4.273969)
+      (xy 4.583406 -4.595437) (xy 5.019969 -4.595437) (xy 5.019969 -4.825625) (xy 5.054695 -5.168922)
+      (xy 5.158875 -5.389187) (xy 5.347391 -5.50825) (xy 5.635125 -5.547937) (xy 5.843484 -5.536031)
+      (xy 6.032 -5.500312) (xy 6.032 -5.174875) (xy 5.722438 -5.230437) (xy 5.547813 -5.198687)
+      (xy 5.476375 -5.065734) (xy 5.461492 -4.929308) (xy 5.456531 -4.722437) (xy 5.456531 -4.595437)
+      (xy 6.032 -4.595437) (xy 6.032 -4.273969) (xy 5.456531 -4.273969) (xy 5.456531 -2.611062)
+      (xy 5.456531 -1.744552) (xy 7.33375 -1.744552) (xy 7.33375 -2.571375) (xy 7.066521 -2.587691)
+      (xy 6.862792 -2.636639) (xy 6.722563 -2.718218) (xy 6.600524 -2.928562) (xy 6.559844 -3.265906)
+      (xy 6.559844 -4.674812) (xy 6.9845 -4.674812) (xy 6.9845 -3.265906) (xy 7.057922 -2.974203)
+      (xy 7.325813 -2.896812) (xy 7.595688 -2.976187) (xy 7.591719 -4.674812) (xy 8.028281 -4.674812)
+      (xy 8.028281 -2.738062) (xy 7.820583 -2.645458) (xy 7.589073 -2.589896) (xy 7.33375 -2.571375)
+      (xy 7.33375 -1.744552) (xy 10.012656 -1.744552) (xy 10.012656 -2.611062) (xy 9.036344 -2.611062)
+      (xy 9.036344 -5.186781) (xy 8.504531 -5.186781) (xy 8.504531 -5.50825) (xy 9.480844 -5.50825)
+      (xy 9.480844 -2.932531) (xy 10.012656 -2.932531) (xy 10.012656 -2.611062) (xy 10.012656 -1.744552)
+      (xy 10.839479 -1.744552) (xy 11.066399 -1.7557) (xy 11.291134 -1.789036) (xy 11.511519 -1.844239)
+      (xy 11.725431 -1.920779) (xy 11.930812 -2.017916) (xy 12.125682 -2.134717) (xy 12.308166 -2.270056)
+      (xy 12.476505 -2.42263) (xy 12.629079 -2.590969) (xy 12.764418 -2.773453) (xy 12.881219 -2.968323)
+      (xy 12.978357 -3.173704) (xy 13.054896 -3.387617) (xy 13.110099 -3.608002) (xy 13.143436 -3.832736)
+      (xy 13.154583 -4.059656) (xy 13.143436 -4.286576) (xy 13.110099 -4.51131) (xy 13.054896 -4.731695)
+      (xy 12.978357 -4.945608) (xy 12.881219 -5.150989) (xy 12.764418 -5.345859) (xy 12.629079 -5.528343)
+      (xy 12.476505 -5.696682) (xy 12.308166 -5.849256) (xy 12.125682 -5.984595) (xy 11.930812 -6.101396)
+      (xy 11.725431 -6.198533) (xy 11.511519 -6.275073) (xy 11.291134 -6.330276) (xy 11.066399 -6.363612)
+      (xy 10.839479 -6.37476) (xy 10.012656 -6.37476) (xy -9.485812 -6.37476)) (layer F.SilkS) (width 0.01))
+  )
   (gr_line (start 51.5 134.5) (end 106.5 134.5) (angle 90) (layer Edge.Cuts) (width 0.15))
